Commit message: Wip on torque control.

File: single_lwr_example/single_lwr_robot/robot/single_lwr_robot.urdf.xacro (robot description, xacro)
@@ -31,5 +31,5 @@
 	<!-- using the models -->
 	<xacro:kuka_lwr parent="box" name="lwr">
-		<origin xyz="0 0 1" rpy="0 0 0"/>
+		<origin xyz="0.77 0.801 1.607" rpy="3.1415 -0.7854 0"/>
 	</xacro:kuka_lwr>
 </robot>
